File: kicad/eel_head_pcbs_assembly/eel_esp32_switch_host_board_v02/eel_esp32_switch_host_board_v02.kicad_sch (KiCad schematic)
At the start: 13 parts, among them J1 Lipo back, J2 motor driver, J3 ELRS RX, J4 Noods front, J5 RGB_DATA, J6 Lipo front, J7 Noods back, Q1 BC817, SW1 SW_Push_DPDT, U1 XIAO-ESP32C3

Commit message: update xiao pcb
Parts:
- C1: value C -> 100nF
